File: can_iface.sch (KiCad schematic (older format))
At the start: 14 parts

Commit message: remove cap from mcp2551
Parts:
- removed C?: C_Small, symbol Device:C_Small
Connections:
- net GND: now also R?.2, U?.2 (VSS)
Changed lines of the file:
@@
 	5400 3950 5400 4100
-Wire Wire Line
-	6100 4700 6100 4950
 Wire Wire Line
 	5400 4300 5400 4450
@@
 	5400 4450 6100 4450
 Connection ~ 6100 4450
-Wire Wire Line
-	6100 4450 6100 4500
 $Comp
 L Connector:Conn_01x03_Female J?
@@
 Text HLabel 3600 5200 1    50   Input ~ 0
 VCC
-$Comp
-L Device:C_Small C?
-U 1 1 61883CD8
-P 6100 4600
-F 0 "C?" H 6192 4646 50  0000 L CNN
-F 1 "C_Small" H 6192 4555 50  0000 L CNN
-F 2 "" H 6100 4600 50  0001 C CNN
-F 3 "~" H 6100 4600 50  0001 C CNN
-	1    6100 4600
-	1    0    0    -1
-$EndComp
+Wire Wire Line
+	6100 4450 6100 4950
 $EndSCHEMATC

Commit message: update reference ids, assign value to c8
Parts:
- gave numbers to parts that had none: 13
Changed lines of the file:
@@
 $EndDescr
 $Comp
-L Interface_CAN_LIN:MCP2515-xSO U?
+L Interface_CAN_LIN:MCP2515-xSO U2
 U 1 1 6187FDDC
 P 3050 4150
-F 0 "U?" H 3050 5131 50  0000 C CNN
+F 0 "U2" H 3050 5131 50  0000 C CNN
 F 1 "MCP2515-xSO" H 3050 5040 50  0000 C CNN
 F 2 "Package_SO:SOIC-18W_7.5x11.6mm_P1.27mm" H 3050 3250 50  0001 C CIN
@@
 $EndComp
 $Comp
-L Interface_CAN_LIN:MCP2551-I-SN U?
+L Interface_CAN_LIN:MCP2551-I-SN U3
 U 1 1 618811D8
 P 6100 3750
-F 0 "U?" H 6100 4331 50  0000 C CNN
+F 0 "U3" H 6100 4331 50  0000 C CNN
 F 1 "MCP2551-I-SN" H 6100 4240 50  0000 C CNN
 F 2 "Package_SO:SOIC-8_3.9x4.9mm_P1.27mm" H 6100 3250 50  0001 C CIN
@@
 	6100 4150 6100 4450
 $Comp
-L Device:R_Small R?
+L Device:R_Small R14
 U 1 1 61884E94
 P 5400 4200
-F 0 "R?" H 5459 4246 50  0000 L CNN
+F 0 "R14" H 5459 4246 50  0000 L CNN
 F 1 "10k" H 5459 4155 50  0000 L CNN
 F 2 "" H 5400 4200 50  0001 C CNN
@@
 Connection ~ 6100 4450
 $Comp
-L Connector:Conn_01x03_Female J?
+L Connector:Conn_01x03_Female J2
 U 1 1 6188C8F1
 P 1150 1350
-F 0 "J?" H 1042 1635 50  0000 C CNN
+F 0 "J2" H 1042 1635 50  0000 C CNN
 F 1 "CAN_CONN" H 1042 1544 50  0000 C CNN
 F 2 "" H 1150 1350 50  0001 C CNN
@@
 	3200 1200 3200 1150
 $Comp
-L Device:Jumper_NO_Small JP?
+L Device:Jumper_NO_Small JP2
 U 1 1 618B011F
 P 3200 1600
-F 0 "JP?" V 3154 1552 50  0000 R CNN
+F 0 "JP2" V 3154 1552 50  0000 R CNN
 F 1 "Jumper" V 3245 1552 50  0000 R CNN
 F 2 "" H 3200 1600 50  0001 C CNN
@@
 $EndComp
 $Comp
-L Device:R_Small R?
+L Device:R_Small R12
 U 1 1 618AFADF
 P 3200 1300
-F 0 "R?" H 3142 1254 50  0000 R CNN
+F 0 "R12" H 3142 1254 50  0000 R CNN
 F 1 "120" H 3142 1345 50  0000 R CNN
 F 2 "" H 3200 1300 50  0001 C CNN
@@
 	2450 3850 1850 3850
 $Comp
-L Device:Crystal_Small Y?
+L Device:Crystal_Small Y1
 U 1 1 618DEC12
 P 1750 4350
-F 0 "Y?" V 1704 4438 50  0000 L CNN
+F 0 "Y1" V 1704 4438 50  0000 L CNN
 F 1 "16MHz" V 1795 4438 50  0000 L CNN
 F 2 "" H 1750 4350 50  0001 C CNN
@@
 $EndComp
 $Comp
-L Device:C_Small C?
+L Device:C_Small C5
 U 1 1 618E0189
 P 1550 4550
-F 0 "C?" V 1321 4550 50  0000 C CNN
+F 0 "C5" V 1321 4550 50  0000 C CNN
 F 1 "22pF" V 1412 4550 50  0000 C CNN
 F 2 "" H 1550 4550 50  0001 C CNN
@@
 	1750 4550 1750 4450
 $Comp
-L Device:C_Small C?
+L Device:C_Small C4
 U 1 1 618E179D
 P 1550 4200
-F 0 "C?" V 1321 4200 50  0000 C CNN
+F 0 "C4" V 1321 4200 50  0000 C CNN
 F 1 "22pF" V 1412 4200 50  0000 C CNN
 F 2 "" H 1550 4200 50  0001 C CNN
@@
 Wire Wire Line
 	5600 3650 3650 3650
-Wire Wire Line
-	7100 3850 6600 3850
-Wire Wire Line
-	7100 3650 6600 3650
 NoConn ~ 5450 3850
 Wire Wire Line
 	5600 3850 5450 3850
 $Comp
-L Device:Jumper_NO_Small JP?
+L Device:Jumper_NO_Small JP3
 U 1 1 6190115F
 P 3950 4150
-F 0 "JP?" H 3950 4335 50  0000 C CNN
+F 0 "JP3" H 3950 4335 50  0000 C CNN
 F 1 "Jumper" H 3950 4244 50  0000 C CNN
 F 2 "" H 3950 4150 50  0001 C CNN
@@
 	4400 4750 4150 4750
 $Comp
-L Device:R_Small R?
+L Device:R_Small R13
 U 1 1 619064FA
 P 4050 4750
-F 0 "R?" V 3854 4750 50  0000 C CNN
+F 0 "R13" V 3854 4750 50  0000 C CNN
 F 1 "10k" V 3945 4750 50  0000 C CNN
 F 2 "" H 4050 4750 50  0001 C CNN
@@
 CAN_INT
 $Comp
-L Device:C_Small C?
+L Device:C_Small C7
 U 1 1 61CFFC49
 P 4000 5400
-F 0 "C?" H 4092 5446 50  0000 L CNN
+F 0 "C7" H 4092 5446 50  0000 L CNN
 F 1 "10uF" H 4092 5355 50  0000 L CNN
 F 2 "" H 4000 5400 50  0001 C CNN
@@
 $EndComp
 $Comp
-L Device:C_Small C?
+L Device:C_Small C6
 U 1 1 61CFFEED
 P 3600 5400
-F 0 "C?" H 3692 5446 50  0000 L CNN
+F 0 "C6" H 3692 5446 50  0000 L CNN
 F 1 "0.1uF" H 3692 5355 50  0000 L CNN
 F 2 "" H 3600 5400 50  0001 C CNN
@@
 Wire Wire Line
 	6100 4450 6100 4950
+Wire Wire Line
+	7100 3850 6600 3850
+Wire Wire Line
+	7100 3650 6600 3650
 $EndSCHEMATC

Commit message: no longer a hat lol
Parts:
- removed J2: CAN_CONN, symbol Connector:Conn_01x03_Female
- added J2: CAN_CON, JST-PH-S4B-K-S-LF-SN:JST_S4B-PH-K-S(LF)(SN), symbol Connector:Conn_01x04_Female
- added TP13, TP14, TP5, TP6: TestPoint, TestPoint:TestPoint_Pad_D2.5mm, symbol Connector:TestPoint
- C4, C5, C6, C7: footprint (none) -> Capacitor_SMD:C_0805_2012Metric_Pad1.15x1.40mm_HandSolder
- JP2, JP3: footprint (none) -> Connector_PinHeader_2.54mm:PinHeader_1x02_P2.54mm_Vertical
- R12, R13, R14: footprint (none) -> Resistor_SMD:R_0805_2012Metric_Pad1.15x1.40mm_HandSolder
- Y1: footprint (none) -> Crystal:Crystal_HC49-U_Vertical
Connections:
- net CAN_H: now also J2.3 (Pin_3), TP13.1
- net CAN_L: now also J2.2 (Pin_2), TP14.1
- net GND: now also J2.1 (Pin_1)
- net at U2.1 (TXCAN), U3.4 (RXD): now also TP6.1
- net at U2.2 (RXCAN), U3.1 (TXD): now also TP5.1
- no-connect marks 7 -> 8
Changed lines of the file:
@@
 F 0 "R14" H 5459 4246 50  0000 L CNN
 F 1 "10k" H 5459 4155 50  0000 L CNN
-F 2 "" H 5400 4200 50  0001 C CNN
+F 2 "Resistor_SMD:R_0805_2012Metric_Pad1.15x1.40mm_HandSolder" H 5400 4200 50  0001 C CNN
 F 3 "~" H 5400 4200 50  0001 C CNN
 	1    5400 4200
@@
 	5400 4450 6100 4450
 Connection ~ 6100 4450
-$Comp
-L Connector:Conn_01x03_Female J2
-U 1 1 6188C8F1
-P 1150 1350
-F 0 "J2" H 1042 1635 50  0000 C CNN
-F 1 "CAN_CONN" H 1042 1544 50  0000 C CNN
-F 2 "" H 1150 1350 50  0001 C CNN
-F 3 "~" H 1150 1350 50  0001 C CNN
-	1    1150 1350
-	-1   0    0    -1
-$EndComp
-Wire Wire Line
-	1350 1450 1550 1450
-Wire Wire Line
-	1550 1450 1550 1650
+Wire Wire Line
+	1300 1600 1500 1600
 Wire Notes Line
 	950  1900 2000 1900
@@
 Text Notes 950  900  0    50   ~ 0
 CAN Connector
-Wire Notes Line
-	2350 950  2350 1900
-Wire Notes Line
-	3350 1900 3350 950
-Wire Notes Line
-	3350 950  2350 950
-Text Notes 2350 900  0    50   ~ 0
-CAN Termination
-Wire Notes Line
-	2350 1900 3350 1900
-Wire Wire Line
-	3200 1750 3200 1700
-Wire Wire Line
-	3200 1400 3200 1500
-Wire Wire Line
-	3200 1200 3200 1150
-$Comp
-L Device:Jumper_NO_Small JP2
-U 1 1 618B011F
-P 3200 1600
-F 0 "JP2" V 3154 1552 50  0000 R CNN
-F 1 "Jumper" V 3245 1552 50  0000 R CNN
-F 2 "" H 3200 1600 50  0001 C CNN
-F 3 "~" H 3200 1600 50  0001 C CNN
-	1    3200 1600
-	0    1    1    0
-$EndComp
-$Comp
-L Device:R_Small R12
-U 1 1 618AFADF
-P 3200 1300
-F 0 "R12" H 3142 1254 50  0000 R CNN
-F 1 "120" H 3142 1345 50  0000 R CNN
-F 2 "" H 3200 1300 50  0001 C CNN
-F 3 "~" H 3200 1300 50  0001 C CNN
-	1    3200 1300
-	1    0    0    1
-$EndComp
 Text HLabel 1850 3750 0    50   Input ~ 0
 SPI_CE0
@@
 F 0 "Y1" V 1704 4438 50  0000 L CNN
 F 1 "16MHz" V 1795 4438 50  0000 L CNN
-F 2 "" H 1750 4350 50  0001 C CNN
+F 2 "Crystal:Crystal_HC49-U_Vertical" H 1750 4350 50  0001 C CNN
 F 3 "~" H 1750 4350 50  0001 C CNN
 	1    1750 4350
@@
 F 0 "C5" V 1321 4550 50  0000 C CNN
 F 1 "22pF" V 1412 4550 50  0000 C CNN
-F 2 "" H 1550 4550 50  0001 C CNN
+F 2 "Capacitor_SMD:C_0805_2012Metric_Pad1.15x1.40mm_HandSolder" H 1550 4550 50  0001 C CNN
 F 3 "~" H 1550 4550 50  0001 C CNN
 	1    1550 4550
@@
 F 0 "C4" V 1321 4200 50  0000 C CNN
 F 1 "22pF" V 1412 4200 50  0000 C CNN
-F 2 "" H 1550 4200 50  0001 C CNN
+F 2 "Capacitor_SMD:C_0805_2012Metric_Pad1.15x1.40mm_HandSolder" H 1550 4200 50  0001 C CNN
 F 3 "~" H 1550 4200 50  0001 C CNN
 	1    1550 4200
@@
 	2550 3350 3050 3350
 Wire Wire Line
-	5600 3550 3650 3550
-Wire Wire Line
-	5600 3650 3650 3650
+	5600 3550 4600 3550
+Wire Wire Line
+	5600 3650 4650 3650
 NoConn ~ 5450 3850
 Wire Wire Line
@@
 F 0 "JP3" H 3950 4335 50  0000 C CNN
 F 1 "Jumper" H 3950 4244 50  0000 C CNN
-F 2 "" H 3950 4150 50  0001 C CNN
+F 2 "Connector_PinHeader_2.54mm:PinHeader_1x02_P2.54mm_Vertical" H 3950 4150 50  0001 C CNN
 F 3 "~" H 3950 4150 50  0001 C CNN
 	1    3950 4150
@@
 F 0 "R13" V 3854 4750 50  0000 C CNN
 F 1 "10k" V 3945 4750 50  0000 C CNN
-F 2 "" H 4050 4750 50  0001 C CNN
+F 2 "Resistor_SMD:R_0805_2012Metric_Pad1.15x1.40mm_HandSolder" H 4050 4750 50  0001 C CNN
 F 3 "~" H 4050 4750 50  0001 C CNN
 	1    4050 4750
@@
 Text Label 7100 3850 2    50   ~ 0
 CAN_L
-Text Label 2650 1150 0    50   ~ 0
+Text Label 1800 1400 2    50   ~ 0
 CAN_H
-Text Label 2600 1750 0    50   ~ 0
+Wire Wire Line
+	1300 1400 1800 1400
+Wire Wire Line
+	1300 1500 1800 1500
+Text Label 1800 1500 2    50   ~ 0
 CAN_L
-Wire Wire Line
-	2600 1750 3200 1750
-Wire Wire Line
-	2650 1150 3200 1150
-Text Label 1850 1250 2    50   ~ 0
-CAN_H
-Wire Wire Line
-	1350 1250 1850 1250
-Wire Wire Line
-	1350 1350 1850 1350
-Text Label 1850 1350 2    50   ~ 0
-CAN_L
-Text HLabel 1550 1650 3    50   Input ~ 0
+Text HLabel 1500 1600 3    50   Input ~ 0
 GND
 Text HLabel 4300 4150 2    50   Input ~ 0
@@
 F 0 "C7" H 4092 5446 50  0000 L CNN
 F 1 "10uF" H 4092 5355 50  0000 L CNN
-F 2 "" H 4000 5400 50  0001 C CNN
+F 2 "Capacitor_SMD:C_0805_2012Metric_Pad1.15x1.40mm_HandSolder" H 4000 5400 50  0001 C CNN
 F 3 "~" H 4000 5400 50  0001 C CNN
 	1    4000 5400
@@
 F 0 "C6" H 3692 5446 50  0000 L CNN
 F 1 "0.1uF" H 3692 5355 50  0000 L CNN
-F 2 "" H 3600 5400 50  0001 C CNN
+F 2 "Capacitor_SMD:C_0805_2012Metric_Pad1.15x1.40mm_HandSolder" H 3600 5400 50  0001 C CNN
 F 3 "~" H 3600 5400 50  0001 C CNN
 	1    3600 5400
@@
 Wire Wire Line
 	7100 3650 6600 3650
+$Comp
+L Connector:Conn_01x04_Female J2
+U 1 1 61A48E3F
+P 1100 1500
+F 0 "J2" H 992 1075 50  0000 C CNN
+F 1 "CAN_CON" H 992 1166 50  0000 C CNN
+F 2 "JST-PH-S4B-K-S-LF-SN:JST_S4B-PH-K-S(LF)(SN)" H 1100 1500 50  0001 C CNN
+F 3 "~" H 1100 1500 50  0001 C CNN
+	1    1100 1500
+	-1   0    0    1
+$EndComp
+NoConn ~ 1300 1300
+$Comp
+L Connector:TestPoint TP5
+U 1 1 61BE96EB
+P 4600 3550
+F 0 "TP5" H 4542 3622 50  0000 R CNN
+F 1 "TestPoint" H 4658 3577 50  0001 L CNN
+F 2 "TestPoint:TestPoint_Pad_D2.5mm" H 4800 3550 50  0001 C CNN
+F 3 "~" H 4800 3550 50  0001 C CNN
+	1    4600 3550
+	-1   0    0    -1
+$EndComp
+Connection ~ 4600 3550
+Wire Wire Line
+	4600 3550 3650 3550
+$Comp
+L Connector:TestPoint TP6
+U 1 1 61BEAEA6
+P 4650 3700
+F 0 "TP6" H 4593 3772 50  0000 R CNN
+F 1 "TestPoint" H 4708 3727 50  0001 L CNN
+F 2 "TestPoint:TestPoint_Pad_D2.5mm" H 4850 3700 50  0001 C CNN
+F 3 "~" H 4850 3700 50  0001 C CNN
+	1    4650 3700
+	1    0    0    1
+$EndComp
+Wire Wire Line
+	4650 3700 4650 3650
+Connection ~ 4650 3650
+Wire Wire Line
+	4650 3650 3650 3650
+Wire Wire Line
+	2650 1150 3200 1150
+Wire Wire Line
+	2600 1750 3200 1750
+Text Label 2600 1750 0    50   ~ 0
+CAN_L
+Text Label 2650 1150 0    50   ~ 0
+CAN_H
+$Comp
+L Device:R_Small R12
+U 1 1 618AFADF
+P 3200 1300
+F 0 "R12" H 3142 1254 50  0000 R CNN
+F 1 "120" H 3142 1345 50  0000 R CNN
+F 2 "Resistor_SMD:R_0805_2012Metric_Pad1.15x1.40mm_HandSolder" H 3200 1300 50  0001 C CNN
+F 3 "~" H 3200 1300 50  0001 C CNN
+	1    3200 1300
+	1    0    0    1
+$EndComp
+$Comp
+L Device:Jumper_NO_Small JP2
+U 1 1 618B011F
+P 3200 1600
+F 0 "JP2" V 3154 1552 50  0000 R CNN
+F 1 "Jumper" V 3245 1552 50  0000 R CNN
+F 2 "Connector_PinHeader_2.54mm:PinHeader_1x02_P2.54mm_Vertical" H 3200 1600 50  0001 C CNN
+F 3 "~" H 3200 1600 50  0001 C CNN
+	1    3200 1600
+	0    1    1    0
+$EndComp
+Wire Wire Line
+	3200 1200 3200 1150
+Wire Wire Line
+	3200 1400 3200 1500
+Wire Wire Line
+	3200 1750 3200 1700
+Wire Notes Line
+	2350 1900 3350 1900
+Text Notes 2350 900  0    50   ~ 0
+CAN Termination
+Wire Notes Line
+	3350 950  2350 950
+Wire Notes Line
+	3350 1900 3350 950
+Wire Notes Line
+	2350 950  2350 1900
+$Comp
+L Connector:TestPoint TP13
+U 1 1 61C5D8AE
+P 7100 3650
+F 0 "TP13" V 7100 3838 50  0000 L CNN
+F 1 "TestPoint" V 7145 3838 50  0001 L CNN
+F 2 "TestPoint:TestPoint_Pad_D2.5mm" H 7300 3650 50  0001 C CNN
+F 3 "~" H 7300 3650 50  0001 C CNN
+	1    7100 3650
+	0    1    1    0
+$EndComp
+$Comp
+L Connector:TestPoint TP14
+U 1 1 61C5E05D
+P 7100 3850
+F 0 "TP14" V 7100 4038 50  0000 L CNN
+F 1 "TestPoint" V 7145 4038 50  0001 L CNN
+F 2 "TestPoint:TestPoint_Pad_D2.5mm" H 7300 3850 50  0001 C CNN
+F 3 "~" H 7300 3850 50  0001 C CNN
+	1    7100 3850
+	0    1    1    0
+$EndComp
 $EndSCHEMATC

Commit message: power supply overhaul
Parts:
- removed R14: 10k, Resistor_SMD:R_0805_2012Metric_Pad1.15x1.40mm_HandSolder, symbol Device:R_Small
- removed TP5, TP6: TestPoint, TestPoint:TestPoint_Pad_D2.5mm, symbol Connector:TestPoint
- removed U2: MCP2515-xSO, Package_SO:SOIC-18W_7.5x11.6mm_P1.27mm, symbol Interface_CAN_LIN:MCP2515-xSO
- removed U3: MCP2551-I-SN, Package_SO:SOIC-8_3.9x4.9mm_P1.27mm, symbol Interface_CAN_LIN:MCP2551-I-SN
- added C7, C8: 0.1uF, Capacitor_SMD:C_0603_1608Metric_Pad1.05x0.95mm_HandSolder, symbol Device:C_Small
- added C9: 1uF, Capacitor_SMD:C_0603_1608Metric_Pad1.05x0.95mm_HandSolder, symbol Device:C_Small
- added U2: MCP2515-xSO, MCP2515-IST:SOP65P640X110-20N, symbol MCP2515:MCP2515-xSO
- added U3: MCP2562-H-MF, MCP2562T-E_SN:SOIC127P600X175-8N, symbol Interface_CAN_LIN:MCP2562-H-MF
- C3: renamed from C4; footprint Capacitor_SMD:C_0805_2012Metric_Pad1.15x1.40mm_HandSolder -> Capacitor_SMD:C_0603_1608Metric_Pad1.05x0.95mm_HandSolder; Description (none) -> 50V MLCC 1%; Manufacturer_Part_Number (none) -> C0603C220F5GACAUTO; category (none) -> CAN; package (none) -> 0603
- C4: renamed from C5; footprint Capacitor_SMD:C_0805_2012Metric_Pad1.15x1.40mm_HandSolder -> Capacitor_SMD:C_0603_1608Metric_Pad1.05x0.95mm_HandSolder; Description (none) -> 50V MLCC 1%; Manufacturer_Part_Number (none) -> C0603C220F5GACAUTO; category (none) -> CAN; package (none) -> 0603
- C5: renamed from C6; footprint Capacitor_SMD:C_0805_2012Metric_Pad1.15x1.40mm_HandSolder -> Capacitor_SMD:C_0603_1608Metric_Pad1.05x0.95mm_HandSolder; Description (none) -> 16V MLCC 10%; Manufacturer_Part_Number (none) -> C0603C104K4RACTU; category (none) -> CAN; package (none) -> 0603
- C6: renamed from C7; footprint Capacitor_SMD:C_0805_2012Metric_Pad1.15x1.40mm_HandSolder -> Capacitor_SMD:C_0603_1608Metric_Pad1.05x0.95mm_HandSolder; Description (none) -> 25V MLCC 10%; Manufacturer_Part_Number (none) -> GRM188R61E106KA73J; category (none) -> CAN; package (none) -> 0603
- J3: renamed from J2; Description (none) -> JST-PH-S4B-K-S-LF-SN JST PH Female; category (none) -> CAN; package (none) -> JST-PH-S4B
- JP2, JP3: Description (none) -> Pin Header; category (none) -> CAN; package (none) -> 2x2.54mm
- R14: renamed from R12; Description (none) -> 100V 125mW Resistor 0.1%; Manufacturer_Part_Number (none) -> ERA-6VEB1200V; category (none) -> CAN; package (none) -> 0805
- R15: renamed from R13; footprint Resistor_SMD:R_0805_2012Metric_Pad1.15x1.40mm_HandSolder -> Resistor_SMD:R_0603_1608Metric_Pad1.05x0.95mm_HandSolder; Description (none) -> 62.5mW Resistor 0.5%; Manufacturer_Part_Number (none) -> CPF0603D10KE; category (none) -> CAN; package (none) -> 0603
- TP6: renamed from TP13; footprint TestPoint:TestPoint_Pad_D2.5mm -> TestPoint:TestPoint_Pad_D1.0mm
- TP7: renamed from TP14; footprint TestPoint:TestPoint_Pad_D2.5mm -> TestPoint:TestPoint_Pad_D1.0mm
- Y1: Description (none) -> 16MHz Crystal Oscillator; Manufacturer_Part_Number (none) -> FC4STCBMF16.0-BAG200; category (none) -> CAN
Connections:
- net CAN_H: now also U3.7 (CANH)
- net CAN_L: now also U3.6 (CANL)
- net GND: now also C7.2, C8.2, C9.2, U2.9 (VSS), U3.2 (VSS), U3.8 (SHDN), U3.9 (PAD)
- net SPI_CE0: now also U2.16 (~CS)
- net SPI_CLK: now also U2.13 (SCK)
- net SPI_MISO: now also U2.15 (SO)
- net SPI_MOSI: now also U2.14 (SI)
- net at JP3.1: now also U2.12 (~INT)
- net at R15.2: now also U2.17 (~RESET)
- net at C3.1, Y1.1: now also U2.7 (OSC2)
- net at C4.2, Y1.2: now also U2.8 (OSC1)
- net VCC renamed Vin_3v3
- net Vin_3v3: now also C7.1, U2.18 (VDD), U3.5 (Vio)
- new net: U2.1 (TXCAN), U3.1 (TXD)
- new net: U2.2 (RXCAN), U3.4 (RXD)
- new net Vin_5v: C8.1, C9.1, U3.3 (VDD)
- no-connect marks 8 -> 7
Other:
- moved on the sheet: TP6, TP7

Commit message: final final sch
Parts:
- U3: value MCP2562-H-MF -> MCP2562-H-P; Manufacturer_Part_Number MCP2562-H-MF -> MCP2562-H-P
Changed lines of the file:
@@
 P 8100 3900
 F 0 "U3" H 8100 4481 50  0000 C CNN
-F 1 "MCP2562-H-MF" H 8100 4390 50  0000 C CNN
+F 1 "MCP2562-H-P" H 8100 4390 50  0000 C CNN
 F 2 "MCP2562T-E_SN:SOIC127P600X175-8N" H 8100 3400 50  0001 C CIN
 F 3 "http://ww1.microchip.com/downloads/en/DeviceDoc/25167A.pdf" H 8100 3900 50  0001 C CNN
 F 4 "MCP2562 CAN Transceiver" H 8100 3900 50  0001 C CNN "Description"
-F 5 "MCP2562-H-MF" H 8100 3900 50  0001 C CNN "Manufacturer_Part_Number"
+F 5 "MCP2562-H-P" H 8100 3900 50  0001 C CNN "Manufacturer_Part_Number"
 F 6 "CAN" H 8100 3900 50  0001 C CNN "category"
 F 7 "SO-8" H 8100 3900 50  0001 C CNN "package"

Commit message: [pcb] added copper planes
Parts:
- J3: footprint JST-PH-S4B-K-S-LF-SN:JST_S4B-PH-K-S(LF)(SN) -> Connector_JST:JST_PH_S4B-PH-SM4-TB_1x04-1MP_P2.00mm_Horizontal
Changed lines of the file:
@@
 F 0 "J3" H 992 1075 50  0000 C CNN
 F 1 "CAN_CON" H 992 1166 50  0000 C CNN
-F 2 "JST-PH-S4B-K-S-LF-SN:JST_S4B-PH-K-S(LF)(SN)" H 1100 1500 50  0001 C CNN
+F 2 "Connector_JST:JST_PH_S4B-PH-SM4-TB_1x04-1MP_P2.00mm_Horizontal" H 1100 1500 50  0001 C CNN
 F 3 "~" H 1100 1500 50  0001 C CNN
 F 4 "JST-PH-S4B-K-S-LF-SN JST PH Female" H 1100 1500 50  0001 C CNN "Description"

Commit message: [rev.2 fixes]  - fix Q4 net pin assignment  - removed UVLO  - fix kelvin connection on R_sense  - fix MCP2515 symbol + pinout  - changed oscillator capacitors for 18uF load capacitance  - PCA9615 biasing resistors
Parts:
- removed U2: MCP2515-xSO, MCP2515-IST:SOP65P640X110-20N, symbol MCP2515:MCP2515-xSO
- added U2: MCP2515-xST, MCP2515-IST:SOP65P640X110-20N, symbol MCP2515:MCP2515-xST
- C3, C4: value 22pF -> 36pF
Changed lines of the file:
@@
 P 1550 4550
 F 0 "C4" V 1321 4550 50  0000 C CNN
-F 1 "22pF" V 1412 4550 50  0000 C CNN
+F 1 "36pF" V 1412 4550 50  0000 C CNN
 F 2 "Capacitor_SMD:C_0603_1608Metric_Pad1.05x0.95mm_HandSolder" H 1550 4550 50  0001 C CNN
 F 3 "~" H 1550 4550 50  0001 C CNN
@@
 P 1550 4200
 F 0 "C3" V 1321 4200 50  0000 C CNN
-F 1 "22pF" V 1412 4200 50  0000 C CNN
+F 1 "36pF" V 1412 4200 50  0000 C CNN
 F 2 "Capacitor_SMD:C_0603_1608Metric_Pad1.05x0.95mm_HandSolder" H 1550 4200 50  0001 C CNN
 F 3 "~" H 1550 4200 50  0001 C CNN
@@
 $EndComp
 $Comp
-L MCP2515:MCP2515-xSO U2
-U 1 1 61C3B8E9
-P 3050 4150
-F 0 "U2" H 3050 5131 50  0000 C CNN
-F 1 "MCP2515-xSO" H 3050 5040 50  0000 C CNN
-F 2 "MCP2515-IST:SOP65P640X110-20N" H 3050 3250 50  0001 C CIN
-F 3 "http://ww1.microchip.com/downloads/en/DeviceDoc/21801e.pdf" H 3150 3350 50  0001 C CNN
-F 4 "MCP2515 CAN Controller" H 3050 4150 50  0001 C CNN "Description"
-F 5 "MCP2515-xSO" H 3050 4150 50  0001 C CNN "Manufacturer_Part_Number"
-F 6 "CAN" H 3050 4150 50  0001 C CNN "category"
-F 7 "SOIC18" H 3050 4150 50  0001 C CNN "package"
-	1    3050 4150
-	1    0    0    -1
-$EndComp
-$Comp
 L Interface_CAN_LIN:MCP2562-H-MF U3
 U 1 1 61C4A7AE
@@
 Wire Wire Line
 	4750 3700 7600 3700
+$Comp
+L MCP2515:MCP2515-xST U2
+U 1 1 61DCB70E
+P 3050 4150
+F 0 "U2" H 3050 5131 50  0000 C CNN
+F 1 "MCP2515-xST" H 3050 5040 50  0000 C CNN
+F 2 "MCP2515-IST:SOP65P640X110-20N" H 3050 3250 50  0001 C CIN
+F 3 "http://ww1.microchip.com/downloads/en/DeviceDoc/21801e.pdf" H 3150 3350 50  0001 C CNN
+	1    3050 4150
+	1    0    0    -1
+$EndComp
 $EndSCHEMATC
