File: diff_i2c.sch (KiCad schematic (older format))
At the start: 16 parts, among them IC1 PCA9615DPJ, J3 SM07B-SRSS-TBLFSN

Commit message: power supply overhaul
Parts:
- C10: renamed from C8; footprint Capacitor_SMD:C_0805_2012Metric_Pad1.15x1.40mm_HandSolder -> Capacitor_SMD:C_0603_1608Metric_Pad1.05x0.95mm_HandSolder; Description (none) -> 25V MLCC 10%; Manufacturer_Part_Number (none) -> GRM188R61E106KA73J; category (none) -> DI2C; package (none) -> 0603
- C11: renamed from C9; footprint Capacitor_SMD:C_0805_2012Metric_Pad1.15x1.40mm_HandSolder -> Capacitor_SMD:C_0603_1608Metric_Pad1.05x0.95mm_HandSolder; Description (none) -> 25V MLCC 10%; Manufacturer_Part_Number (none) -> GRM188R61E106KA73J; category (none) -> EEPROM; package (none) -> 0603
- C12: renamed from C10; footprint Capacitor_SMD:C_0805_2012Metric_Pad1.15x1.40mm_HandSolder -> Capacitor_SMD:C_0603_1608Metric_Pad1.05x0.95mm_HandSolder; Description (none) -> 25V MLCC 10%; Manufacturer_Part_Number (none) -> GRM188R61E106KA73J; category (none) -> EEPROM; package (none) -> 0603
- IC1: category (none) -> DI2C; package (none) -> 10-MSOP
- J4: renamed from J3; Description (none) -> JST-SM Connector 7 Position; Manufacturer_Part_Number (none) -> SM07B-SRSS-TBLFSN
- JP4, JP5, JP6: Description (none) -> Pin Header; category (none) -> DI2C; package (none) -> 2x2.54mm
- R16: renamed from R15; Description (none) -> 100V 125mW Resistor 0.1%; Manufacturer_Part_Number (none) -> ERA-6VEB1200V; category (none) -> DI2C; package (none) -> 0805
- R17: renamed from R16; Description (none) -> 100V 125mW Resistor 0.1%; Manufacturer_Part_Number (none) -> ERA-6VEB1200V; category (none) -> DI2C; package (none) -> 0805
- TP10: renamed from TP9; footprint TestPoint:TestPoint_Pad_D2.5mm -> TestPoint:TestPoint_Pad_D1.0mm
- TP11: renamed from TP10; footprint TestPoint:TestPoint_Pad_D2.5mm -> TestPoint:TestPoint_Pad_D1.0mm
- TP12: renamed from TP11; footprint TestPoint:TestPoint_Pad_D2.5mm -> TestPoint:TestPoint_Pad_D1.0mm
- TP13: renamed from TP12; footprint TestPoint:TestPoint_Pad_D2.5mm -> TestPoint:TestPoint_Pad_D1.0mm
- TP8: renamed from TP7; footprint TestPoint:TestPoint_Pad_D2.5mm -> TestPoint:TestPoint_Pad_D1.0mm
- TP9: renamed from TP8; footprint TestPoint:TestPoint_Pad_D2.5mm -> TestPoint:TestPoint_Pad_D1.0mm
Changed lines of the file:
@@
 $Descr A4 11693 8268
 encoding utf-8
-Sheet 3 8
+Sheet 3 7
 Title ""
 Date ""
@@
 $EndDescr
 $Comp
-L JST-SM07B-SRSS-TB:SM07B-SRSS-TBLFSN J3
+L JST-SM07B-SRSS-TB:SM07B-SRSS-TBLFSN J4
 U 1 1 61968298
 P 1600 1300
-F 0 "J3" H 1208 1665 50  0000 C CNN
+F 0 "J4" H 1208 1665 50  0000 C CNN
 F 1 "SM07B-SRSS-TBLFSN" H 1208 1574 50  0000 C CNN
 F 2 "SM07B-SRSS-TB:JST-SM07B-SRSS-TBLFSN-0" H 1600 1800 50  0001 L CNN
@@
 F 18 "+85°C" H 1600 3400 50  0001 L CNN "temperature range high"
 F 19 "-25°C" H 1600 3500 50  0001 L CNN "temperature range low"
+F 20 "JST-SM Connector 7 Position" H 1600 1300 50  0001 C CNN "Description"
+F 21 "SM07B-SRSS-TBLFSN" H 1600 1300 50  0001 C CNN "Manufacturer_Part_Number"
 	1    1600 1300
 	1    0    0    -1
@@
 F 2 "Connector_PinHeader_2.54mm:PinHeader_1x02_P2.54mm_Vertical" H 2000 2700 50  0001 C CNN
 F 3 "~" H 2000 2700 50  0001 C CNN
+F 4 "Pin Header" H 2000 2700 50  0001 C CNN "Description"
+F 5 "DI2C" H 2000 2700 50  0001 C CNN "category"
+F 6 "2x2.54mm" H 2000 2700 50  0001 C CNN "package"
 	1    2000 2700
 	0    -1   -1   0
@@
 	2000 2500 2400 2500
 $Comp
-L Device:C_Small C8
+L Device:C_Small C10
 U 1 1 6196BE9A
 P 2000 3100
-F 0 "C8" H 2092 3146 50  0000 L CNN
+F 0 "C10" H 2092 3146 50  0000 L CNN
 F 1 "10uF" H 2092 3055 50  0000 L CNN
-F 2 "Capacitor_SMD:C_0805_2012Metric_Pad1.15x1.40mm_HandSolder" H 2000 3100 50  0001 C CNN
+F 2 "Capacitor_SMD:C_0603_1608Metric_Pad1.05x0.95mm_HandSolder" H 2000 3100 50  0001 C CNN
 F 3 "~" H 2000 3100 50  0001 C CNN
+F 4 "25V MLCC 10%" H 2000 3100 50  0001 C CNN "Description"
+F 5 "GRM188R61E106KA73J" H 2000 3100 50  0001 C CNN "Manufacturer_Part_Number"
+F 6 "DI2C" H 2000 3100 50  0001 C CNN "category"
+F 7 "0603" H 2000 3100 50  0001 C CNN "package"
 	1    2000 3100
 	1    0    0    -1
@@
 F 8 "1.1mm" H 5450 3550 50  0001 L BNN "Height"
 F 9 "771-PCA9615DPJ" H 5450 3550 50  0001 L BNN "Mouser_Part_Number"
+F 10 "DI2C" H 5450 3550 50  0001 C CNN "category"
+F 11 "10-MSOP" H 5450 3550 50  0001 C CNN "package"
 	1    5450 3550
 	1    0    0    -1
@@
 	5450 3150 5450 3550
 $Comp
-L Device:C_Small C10
+L Device:C_Small C12
 U 1 1 6198DB03
 P 4300 4200
-F 0 "C10" H 4392 4246 50  0000 L CNN
+F 0 "C12" H 4392 4246 50  0000 L CNN
 F 1 "10uF" H 4392 4155 50  0000 L CNN
-F 2 "Capacitor_SMD:C_0805_2012Metric_Pad1.15x1.40mm_HandSolder" H 4300 4200 50  0001 C CNN
+F 2 "Capacitor_SMD:C_0603_1608Metric_Pad1.05x0.95mm_HandSolder" H 4300 4200 50  0001 C CNN
 F 3 "~" H 4300 4200 50  0001 C CNN
+F 4 "25V MLCC 10%" H 4300 4200 50  0001 C CNN "Description"
+F 5 "GRM188R61E106KA73J" H 4300 4200 50  0001 C CNN "Manufacturer_Part_Number"
+F 6 "EEPROM" H 4300 4200 50  0001 C CNN "category"
+F 7 "0603" H 4300 4200 50  0001 C CNN "package"
 	1    4300 4200
 	1    0    0    -1
@@
 	4300 4300 4300 4400
 $Comp
-L Device:C_Small C9
+L Device:C_Small C11
 U 1 1 61991791
 P 3900 4200
-F 0 "C9" H 3992 4246 50  0000 L CNN
+F 0 "C11" H 3992 4246 50  0000 L CNN
 F 1 "10uF" H 3992 4155 50  0000 L CNN
-F 2 "Capacitor_SMD:C_0805_2012Metric_Pad1.15x1.40mm_HandSolder" H 3900 4200 50  0001 C CNN
+F 2 "Capacitor_SMD:C_0603_1608Metric_Pad1.05x0.95mm_HandSolder" H 3900 4200 50  0001 C CNN
 F 3 "~" H 3900 4200 50  0001 C CNN
+F 4 "25V MLCC 10%" H 3900 4200 50  0001 C CNN "Description"
+F 5 "GRM188R61E106KA73J" H 3900 4200 50  0001 C CNN "Manufacturer_Part_Number"
+F 6 "EEPROM" H 3900 4200 50  0001 C CNN "category"
+F 7 "0603" H 3900 4200 50  0001 C CNN "package"
 	1    3900 4200
 	1    0    0    -1
@@
 F 2 "Connector_PinHeader_2.54mm:PinHeader_1x02_P2.54mm_Vertical" H 1600 4600 50  0001 C CNN
 F 3 "~" H 1600 4600 50  0001 C CNN
+F 4 "Pin Header" H 1600 4600 50  0001 C CNN "Description"
+F 5 "DI2C" H 1600 4600 50  0001 C CNN "category"
+F 6 "2x2.54mm" H 1600 4600 50  0001 C CNN "package"
 	1    1600 4600
 	0    1    1    0
@@
 P 1600 4900
 AR Path="/6187FA0A/61A1282F" Ref="R?"  Part="1"
-AR Path="/6195FE87/61A1282F" Ref="R15"  Part="1"
-F 0 "R15" H 1542 4854 50  0000 R CNN
+AR Path="/6195FE87/61A1282F" Ref="R16"  Part="1"
+F 0 "R16" H 1542 4854 50  0000 R CNN
 F 1 "120" H 1542 4945 50  0000 R CNN
 F 2 "Resistor_SMD:R_0805_2012Metric_Pad1.15x1.40mm_HandSolder" H 1600 4900 50  0001 C CNN
 F 3 "~" H 1600 4900 50  0001 C CNN
+F 4 "100V 125mW Resistor 0.1%" H 1600 4900 50  0001 C CNN "Description"
+F 5 "ERA-6VEB1200V" H 1600 4900 50  0001 C CNN "Manufacturer_Part_Number"
+F 6 "DI2C" H 1600 4900 50  0001 C CNN "category"
+F 7 "0805" H 1600 4900 50  0001 C CNN "package"
 	1    1600 4900
 	1    0    0    1
@@
 F 2 "Connector_PinHeader_2.54mm:PinHeader_1x02_P2.54mm_Vertical" H 2250 4600 50  0001 C CNN
 F 3 "~" H 2250 4600 50  0001 C CNN
+F 4 "Pin Header" H 2250 4600 50  0001 C CNN "Description"
+F 5 "DI2C" H 2250 4600 50  0001 C CNN "category"
+F 6 "2x2.54mm" H 2250 4600 50  0001 C CNN "package"
 	1    2250 4600
 	0    1    1    0
@@
 P 2250 4900
 AR Path="/6187FA0A/61A23D41" Ref="R?"  Part="1"
-AR Path="/6195FE87/61A23D41" Ref="R16"  Part="1"
-F 0 "R16" H 2192 4854 50  0000 R CNN
+AR Path="/6195FE87/61A23D41" Ref="R17"  Part="1"
+F 0 "R17" H 2192 4854 50  0000 R CNN
 F 1 "120" H 2192 4945 50  0000 R CNN
 F 2 "Resistor_SMD:R_0805_2012Metric_Pad1.15x1.40mm_HandSolder" H 2250 4900 50  0001 C CNN
 F 3 "~" H 2250 4900 50  0001 C CNN
+F 4 "100V 125mW Resistor 0.1%" H 2250 4900 50  0001 C CNN "Description"
+F 5 "ERA-6VEB1200V" H 2250 4900 50  0001 C CNN "Manufacturer_Part_Number"
+F 6 "DI2C" H 2250 4900 50  0001 C CNN "category"
+F 7 "0805" H 2250 4900 50  0001 C CNN "package"
 	1    2250 4900
 	1    0    0    1
@@
 	6750 3650 7050 3650
 $Comp
-L Connector:TestPoint TP9
+L Connector:TestPoint TP10
 U 1 1 61B8A771
 P 7050 3650
-F 0 "TP9" V 7050 3838 50  0000 L CNN
+F 0 "TP10" V 7050 3838 50  0000 L CNN
 F 1 "TestPoint" V 7095 3838 50  0001 L CNN
-F 2 "TestPoint:TestPoint_Pad_D2.5mm" H 7250 3650 50  0001 C CNN
+F 2 "TestPoint:TestPoint_Pad_D1.0mm" H 7250 3650 50  0001 C CNN
 F 3 "~" H 7250 3650 50  0001 C CNN
 	1    7050 3650
@@
 $EndComp
 $Comp
-L Connector:TestPoint TP10
+L Connector:TestPoint TP11
 U 1 1 61B8ADC9
 P 7050 3750
-F 0 "TP10" V 7050 3938 50  0000 L CNN
+F 0 "TP11" V 7050 3938 50  0000 L CNN
 F 1 "TestPoint" V 7095 3938 50  0001 L CNN
-F 2 "TestPoint:TestPoint_Pad_D2.5mm" H 7250 3750 50  0001 C CNN
+F 2 "TestPoint:TestPoint_Pad_D1.0mm" H 7250 3750 50  0001 C CNN
 F 3 "~" H 7250 3750 50  0001 C CNN
 	1    7050 3750
@@
 $EndComp
 $Comp
-L Connector:TestPoint TP11
+L Connector:TestPoint TP12
 U 1 1 61B8C5BF
 P 7050 3850
-F 0 "TP11" V 7050 4038 50  0000 L CNN
+F 0 "TP12" V 7050 4038 50  0000 L CNN
 F 1 "TestPoint" V 7095 4038 50  0001 L CNN
-F 2 "TestPoint:TestPoint_Pad_D2.5mm" H 7250 3850 50  0001 C CNN
+F 2 "TestPoint:TestPoint_Pad_D1.0mm" H 7250 3850 50  0001 C CNN
 F 3 "~" H 7250 3850 50  0001 C CNN
 	1    7050 3850
@@
 $EndComp
 $Comp
-L Connector:TestPoint TP12
+L Connector:TestPoint TP13
 U 1 1 61B8C5C5
 P 7050 3950
-F 0 "TP12" V 7050 4138 50  0000 L CNN
+F 0 "TP13" V 7050 4138 50  0000 L CNN
 F 1 "TestPoint" V 7095 4138 50  0001 L CNN
-F 2 "TestPoint:TestPoint_Pad_D2.5mm" H 7250 3950 50  0001 C CNN
+F 2 "TestPoint:TestPoint_Pad_D1.0mm" H 7250 3950 50  0001 C CNN
 F 3 "~" H 7250 3950 50  0001 C CNN
 	1    7050 3950
@@
 	1500 2300 3050 2300
 $Comp
-L Connector:TestPoint TP8
+L Connector:TestPoint TP9
 U 1 1 61B915B9
 P 3050 2400
-F 0 "TP8" H 2992 2426 50  0000 R CNN
+F 0 "TP9" H 2992 2426 50  0000 R CNN
 F 1 "TestPoint" H 2992 2517 50  0000 R CNN
-F 2 "TestPoint:TestPoint_Pad_D2.5mm" H 3250 2400 50  0001 C CNN
+F 2 "TestPoint:TestPoint_Pad_D1.0mm" H 3250 2400 50  0001 C CNN
 F 3 "~" H 3250 2400 50  0001 C CNN
 	1    3050 2400
@@
 	3050 2300 3250 2300
 $Comp
-L Connector:TestPoint TP7
+L Connector:TestPoint TP8
 U 1 1 61B932FB
 P 3050 2100
-F 0 "TP7" H 3108 2172 50  0000 L CNN
+F 0 "TP8" H 3108 2172 50  0000 L CNN
 F 1 "TestPoint" H 3108 2127 50  0001 L CNN
-F 2 "TestPoint:TestPoint_Pad_D2.5mm" H 3250 2100 50  0001 C CNN
+F 2 "TestPoint:TestPoint_Pad_D1.0mm" H 3250 2100 50  0001 C CNN
 F 3 "~" H 3250 2100 50  0001 C CNN
 	1    3050 2100
